Commit message: latest update - robot _hardwre

File: src/robot_desc/urdf/diff_robot.urdf (robot description, URDF)
Before this commit: robot patrol_robot, 9 links, 8 joints
Links:
- removed link wheel_left
- removed link wheel_right
- added link left_wheel, mass 0.75; collision cylinder length=0.04 radius=0.06858; visual cylinder length=0.04 radius=0.06858
- added link right_wheel, mass 0.75; collision cylinder length=0.04 radius=0.06858; visual cylinder length=0.04 radius=0.06858
Joints:
- removed joint wheel_left_joint
- removed joint wheel_right_joint
- added joint left_wheel_joint: type continuous, parent base_link, child left_wheel, origin xyz=0.042 -0.16 0.04 rpy=1.5708 0.0 3.14, axis 0.0 0 1
- added joint right_wheel_joint: type continuous, parent base_link, child right_wheel, origin xyz=0.042 0.16 0.04   rpy=1.5708 0.0 0.0, axis 0.0 0 1

Commit message: see changes being made

File: src/robot_desc/urdf/diff_robot.urdf (robot description, URDF)
Before this commit: robot patrol_robot, 9 links, 8 joints
Joints:
- joint caster_joint: type continuous -> fixed
- joint left_wheel_joint: type continuous -> fixed
- joint right_wheel_joint: type continuous -> fixed

File: src/robot_desc/urdf/ros2_control.xacro (robot description, xacro)
@@ -1,43 +1,48 @@
 <?xml version="1.0"?>
-<robot xmlns:xacro="http://www.ros.org/wiki/xacro" >
-    <ros2_control name="robot_hardware" type="system">
-        <hardware>
-            <plugin>robot_hardware/DiffDriveArduinoHardware</plugin>
-                <param name="left_wheel_name">left_wheel_joint</param>
-                <param name="right_wheel_name">right_wheel_joint</param>
-                <param name="loop_rate">30</param>
-                <param name="device">/dev/ttyUSB0</param>
-                <param name="baud_rate">9600</param>
-        </hardware>
-        <joint name="left_wheel_joint">
-            <command_interface name="velocity"/>
-            <state_interface name="position"/>
-            <state_interface name="velocity"/>
-        </joint>
-        <joint name="right_wheel_joint">
-            <command_interface name="velocity"/>
-            <state_interface name="position"/>
-            <state_interface name="velocity"/>
-        </joint>
-    </ros2_control>
-        <transmission name="left_wheel_trans">
-        <type>transmission_interface/SimpleTransmission</type>
-        <joint name="left_wheel_joint">
-        <hardwareInterface>hardware_interface/VelocityJointInterface</hardwareInterface>
-        </joint>
-        <actuator name="left_wheel_motor">
-        <hardwareInterface>hardware_interface/VelocityJointInterface</hardwareInterface>
-        <mechanicalReduction>1</mechanicalReduction>
-        </actuator>
-    </transmission>
-    <transmission name="right_wheel_trans">
-        <type>transmission_interface/SimpleTransmission</type>
-        <joint name="right_wheel_joint">
-        <hardwareInterface>hardware_interface/VelocityJointInterface</hardwareInterface>
-        </joint>
-        <actuator name="right_wheel_motor">
-        <hardwareInterface>hardware_interface/VelocityJointInterface</hardwareInterface>
-        <mechanicalReduction>1</mechanicalReduction>
-        </actuator>
-    </transmission>
+<robot xmlns:xacro="http://www.ros.org/wiki/xacro">
+  <ros2_control name="robot_hardware" type="system">
+    <hardware>
+      <plugin>robot_hardware/DiffDriveArduinoHardware</plugin>
+        <param name="left_wheel_name">left_wheel_joint</param>
+        <param name="right_wheel_name">right_wheel_joint</param>
+        <param name="loop_rate">"30"</param>
+        <param name="device">"/dev/ttyUSB0"</param>
+        <param name="device">"/dev/ttyUSB0"</param>
+        <param name="baud_rate">"9600"</param>
+        <param name="enc_counts_per_rev">"360"</param>
+        <param name="wheel_radius">"0.05"</param>
+        <param name="wheel_separation">"0.2"</param>
+        <param name="timeout">"0.5"</param>
+    </hardware>
+    <joint name="left_wheel_joint">
+      <command_interface name="velocity"/>
+      <state_interface name="position"/>
+      <state_interface name="velocity"/>
+    </joint>
+    <joint name="right_wheel_joint">
+      <command_interface name="velocity"/>
+      <state_interface name="position"/>
+      <state_interface name="velocity"/>
+    </joint>
+  </ros2_control>
+  <transmission name="left_wheel_trans">
+    <type>transmission_interface/SimpleTransmission</type>
+    <joint name="left_wheel_joint">
+      <hardwareInterface>hardware_interface/VelocityJointInterface</hardwareInterface>
+    </joint>
+    <actuator name="left_wheel_motor">
+      <hardwareInterface>hardware_interface/VelocityJointInterface</hardwareInterface>
+      <mechanicalReduction>1</mechanicalReduction>
+    </actuator>
+  </transmission>
+  <transmission name="right_wheel_trans">
+    <type>transmission_interface/SimpleTransmission</type>
+    <joint name="right_wheel_joint">
+      <hardwareInterface>hardware_interface/VelocityJointInterface</hardwareInterface>
+    </joint>
+    <actuator name="right_wheel_motor">
+      <hardwareInterface>hardware_interface/VelocityJointInterface</hardwareInterface>
+      <mechanicalReduction>1</mechanicalReduction>
+    </actuator>
+  </transmission>
 </robot>

Commit message: Initial commit

File: src/robot_desc/urdf/diff_robot.urdf (robot description, URDF)
Before this commit: robot patrol_robot, 9 links, 8 joints
Joints:
- joint left_wheel_joint: type fixed -> continuous
- joint right_wheel_joint: type fixed -> continuous

File: src/robot_desc/urdf/ros2_control.xacro (robot description, xacro)
@@ -6,12 +6,11 @@
         <param name="left_wheel_name">left_wheel_joint</param>
         <param name="right_wheel_name">right_wheel_joint</param>
-        <param name="loop_rate">"30"</param>
+        <param name="loop_rate">30</param>
         <param name="device">"/dev/ttyUSB0"</param>
-        <param name="device">"/dev/ttyUSB0"</param>
-        <param name="baud_rate">"9600"</param>
-        <param name="enc_counts_per_rev">"360"</param>
-        <param name="wheel_radius">"0.05"</param>
-        <param name="wheel_separation">"0.2"</param>
-        <param name="timeout">"0.5"</param>
+        <param name="baud_rate">9600</param>
+        <param name="enc_counts_per_rev">360</param>
+        <param name="wheel_radius">0.05</param>
+        <param name="wheel_separation">0.2</param>
+        <param name="timeout">0.5</param>
     </hardware>
     <joint name="left_wheel_joint">

Commit message: First upload

File: src/robot_desc/urdf/diff_robot.urdf (robot description, URDF)
Before this commit: robot patrol_robot, 9 links, 8 joints
Links:
- link base_link: mass 2 -> 5
- link caster: geometry collision sphere radius=0.04; visual mesh filename=package://robot_desc/meshes/front_caster.stl
Joints:
- joint base_joint: origin xyz=0 0 0.04 rpy=0 0 0 -> xyz=0 0 0.06858 rpy=0 0 0
- joint caster_joint: origin xyz=-0.0635 0 -0.01 rpy=0.0 0.0 0.0 -> xyz=-0.2 0 -0.03 rpy=0.0 0.0 0.0
- joint left_wheel_joint: origin xyz=0.042 -0.16 0.04 rpy=1.5708 0.0 3.14 -> xyz=0.042 0.16 0.0 rpy=1.5708 0.0 0.0
- joint right_wheel_joint: origin xyz=0.042 0.16 0.04   rpy=1.5708 0.0 0.0 -> xyz=0.042 -0.16 0.0 rpy=1.5708 0.0 0.0
- joint weight_joint: parent base_footprint -> base_link

Commit message: feat: full workspace sync with physical scripts and config

File: src/robot_desc/urdf/diff_robot.urdf (robot description, URDF)
Before this commit: robot patrol_robot, 9 links, 8 joints
Links:
- link base_link: mass 5 -> 2
- link caster: geometry collision mesh filename=package://robot_desc/meshes/front_caster.stl; collision sphere radius=0.04
Joints:
- joint base_joint: origin xyz=0 0 0.06858 rpy=0 0 0 -> xyz=0 0 0.04 rpy=0 0 3.14159
- joint caster_joint: origin xyz=-0.2 0 -0.03 rpy=0.0 0.0 0.0 -> xyz=0.3 0 0 rpy=0.0 0.0 0.0; type fixed -> continuous
- joint left_wheel_joint: origin xyz=0.042 0.16 0.0 rpy=1.5708 0.0 0.0 -> xyz=0.042 -0.16 0.04 rpy=1.5708 0.0 0.0
- joint right_wheel_joint: origin xyz=0.042 -0.16 0.0 rpy=1.5708 0.0 0.0 -> xyz=0.042 0.16 0.04   rpy=1.5708 0.0 0.0
- joint weight_joint: parent base_link -> base_footprint
